Commit message: Fixed sensor name

File: models/simply_diff_drive_robot/simply_diff_drive_robot.urdf (robot description, URDF)
Before this commit: robot diff_bot, 11 links, 10 joints
Links:
- removed link 3d_laser_scanner
- added link lidar, mass 0.3; collision cylinder length=0.13 radius=0.06; visual cylinder length=0.1 radius=0.06
Joints:
- joint 3d_laser_scanner_joint: child 3d_laser_scanner -> lidar

Commit message: Support slip

File: models/simply_diff_drive_robot/simply_diff_drive_robot.urdf (robot description, URDF)
Before this commit: robot diff_bot, 11 links, 10 joints
Joints:
- joint front_free_wheel_base_joint: limit lower=-1e16 upper=1e16 effort=0 velocity=0 -> lower=-1e16 upper=1e16 effort=0 velocity=16
- joint front_free_wheel_joint: limit lower=-1e16 upper=1e16 effort=0 velocity=0 -> lower=-1e16 upper=1e16 effort=0 velocity=16
- joint left_motor_joint: limit lower=-1e16 upper=1e16 effort=0.5 velocity=8 -> lower=-1e16 upper=1e16 effort=3.5 velocity=8
- joint right_motor_joint: limit lower=-1e16 upper=1e16 effort=0.5 velocity=8 -> lower=-1e16 upper=1e16 effort=3.5 velocity=8

Commit message: Support humble

File: models/simply_diff_drive_robot/simply_diff_drive_robot.urdf (robot description, URDF)
Before this commit: robot diff_bot, 11 links, 10 joints
Joints:
- joint front_free_wheel_base_joint: limit lower=-1e16 upper=1e16 effort=0 velocity=0 -> lower=-1e16 upper=1e16 effort=1e1 velocity=1e3
- joint front_free_wheel_joint: limit lower=-1e16 upper=1e16 effort=0 velocity=0 -> lower=-1e16 upper=1e16 effort=1e1 velocity=1e3
- joint left_motor_joint: limit lower=-1e16 upper=1e16 effort=0.5 velocity=8 -> lower=-1e16 upper=1e16 effort=3.5 velocity=8
- joint right_motor_joint: limit lower=-1e16 upper=1e16 effort=0.5 velocity=8 -> lower=-1e16 upper=1e16 effort=3.5 velocity=8
